File: hw/sch_pcb/TFGPSLITE02.kicad_sch (KiCad schematic)
At the start: 26 parts, among them IC1 CAM-M8Q, J1 SM06B-GHS-TB, J2 SM04B-GHS-TB, M1 HOLE, M2 HOLE, M3 HOLE, M4 HOLE, U1 MIC5504-3.3YM5

Commit message: Design of TFGPSLITE01
Parts:
- removed IC1: CAM-M8Q, Mlab_IO:CAM-M8Q, symbol MLAB_IO:CAM-M8Q
- added U2: SAM-M8Q, RF_GPS:ublox_SAM-M8Q, symbol RF_GPS:SAM-M8Q
Connections:
- net +3V3: now also U2.17 (VCC), U2.2 (VCC_IO)
- net EXTINT: now also U2.19 (EXTINT)
- net GND: now also U2.1 (GND), U2.10 (GND), U2.11 (GND), U2.15 (GND), U2.16 (GND), U2.20 (GND), U2.4 (GND), U2.5 (GND), U2.6 (GND)
- net L_UBX_RX: now also U2.14 (RXD)
- net L_UBX_TX: now also U2.13 (TXD)
- net TPL: now also U2.7 (TIMEPULSE)
- net UBX_VBCKP: now reaches C2.1, D1.1 (K)
- net UBX_VBCKP: now also U2.3 (V_BCKP)
- net at R6.2: now also U2.12 (SCL)
- net at R5.2: now also U2.9 (SDA)
- no-connect marks 6 -> 2
Other:
- moved on the sheet: R3, R5, R6

Commit message: improve layout
Parts:
- added C5: 100n, Capacitor_SMD:C_0805_2012Metric, symbol Device:C_Small
Connections:
- net +3V3: now also C5.1
- net GND: now also C5.2
Changed lines of the file:
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@@
+	)
+	(junction
+		(at 144.78 29.21)
+		(diameter 0)
+		(color 0 0 0 0)
 	)
 	(junction
@@
 	(wire
 		(pts
-			(xy 137.16 29.21) (xy 153.67 29.21)
+			(xy 137.16 29.21) (xy 144.78 29.21)
 		)
 		(stroke
@@
 	(wire
 		(pts
+			(xy 144.78 36.83) (xy 144.78 39.37)
+		)
+		(stroke
+			(width 0)
+			(type default)
+		)
+	)
+	(wire
+		(pts
+			(xy 144.78 29.21) (xy 153.67 29.21)
+		)
+		(stroke
+			(width 0)
+			(type default)
+		)
+	)
+	(wire
+		(pts
 			(xy 105.41 29.21) (xy 110.49 29.21)
 		)
@@
 		(pts
 			(xy 170.18 132.08) (xy 158.75 132.08)
+		)
+		(stroke
+			(width 0)
+			(type default)
+		)
+	)
+	(wire
+		(pts
+			(xy 144.78 31.75) (xy 144.78 29.21)
 		)
 		(stroke
@@
 		(on_board yes)
 		(dnp no)
-		(fields_autoplaced yes)
 		(property "Reference" "C4"
 			(at 139.7 33.0262 0)
@@
 		)
 		(property "Value" "100n"
-			(at 139.7 35.5662 0)
+			(at 137.668 36.576 0)
 			(effects
 				(font
@@
 	(symbol
 		(lib_id "power:GND")
+		(at 144.78 39.37 0)
+		(unit 1)
+		(exclude_from_sim no)
+		(in_bom yes)
+		(on_board yes)
+		(dnp no)
+		(fields_autoplaced yes)
+		(property "Reference" "#PWR03"
+			(at 144.78 45.72 0)
+			(effects
+				(font
+					(size 1.27 1.27)
+				)
+				(hide yes)
+			)
+		)
+		(property "Value" "GND"
+			(at 144.78 44.45 0)
+			(effects
+				(font
+					(size 1.27 1.27)
+				)
+			)
+		)
+		(property "Footprint" ""
+			(at 144.78 39.37 0)
+			(effects
+				(font
+					(size 1.27 1.27)
+				)
+				(hide yes)
+			)
+		)
+		(property "Datasheet" ""
+			(at 144.78 39.37 0)
+			(effects
+				(font
+					(size 1.27 1.27)
+				)
+				(hide yes)
+			)
+		)
+		(property "Description" "Power symbol creates a global label with name \"GND\" , ground"
+			(at 144.78 39.37 0)
+			(effects
+				(font
+					(size 1.27 1.27)
+				)
+				(hide yes)
+			)
+		)
+		(pin "1"
+		)
+		(instances
+			(project "TFGPSLITE02"
+				(path "/ad3de673-2c6f-49c5-bb76-b63aef50b486"
+					(reference "#PWR03")
+					(unit 1)
+				)
+			)
+		)
+	)
+	(symbol
+		(lib_id "power:GND")
 		(at 137.16 39.37 0)
 		(unit 1)
@@
 					(unit 1)
 				)
+			)
+		)
+	)
+	(symbol
+		(lib_id "Device:C_Small")
+		(at 144.78 34.29 0)
+		(unit 1)
+		(exclude_from_sim no)
+		(in_bom yes)
+		(on_board yes)
+		(dnp no)
+		(fields_autoplaced yes)
+		(property "Reference" "C5"
+			(at 147.32 33.0262 0)
+			(effects
+				(font
+					(size 1.27 1.27)
+				)
+				(justify left)
+			)
+		)
+		(property "Value" "100n"
+			(at 147.32 35.5662 0)
+			(effects
+				(font
+					(size 1.27 1.27)
+				)
+				(justify left)
+			)
+		)
+		(property "Footprint" "Capacitor_SMD:C_0805_2012Metric"
+			(at 144.78 34.29 0)
+			(effects
+				(font
+					(size 1.27 1.27)
+				)
+				(hide yes)
+			)
+		)
+		(property "Datasheet" "~"
+			(at 144.78 34.29 0)
+			(effects
+				(font
+					(size 1.27 1.27)
+				)
+				(hide yes)
+			)
+		)
+		(property "Description" "Unpolarized capacitor, small symbol"
+			(at 144.78 34.29 0)
+			(effects
+				(font
+					(size 1.27 1.27)
+				)
+				(hide yes)
+			)
+		)
+		(property "UST_ID" "5c70984812875079b91f8bf2"
+			(at 144.78 34.29 0)
+			(effects
+				(font
+					(size 1.27 1.27)
+				)
+				(hide yes)
+			)
+		)
+		(pin "1"
+		)
+		(pin "2"
+		)
+		(instances
+			(project "TFGPSLITE02"
+				(path "/ad3de673-2c6f-49c5-bb76-b63aef50b486"
+					(reference "C5")
+					(unit 1)
+				)
