File: hw/sch_pcb/TFGPSLITE02.kicad_pcb (KiCad board)
At the start: 2 copper layers, 50 x 50 mm, 26 parts, among them J1 SM06B-GHS-TB, J2 SM04B-GHS-TB, M1 HOLE, M2 HOLE, M3 HOLE, M4 HOLE, U1 MIC5504-3.3YM5, U2 SAM-M8Q

Commit message: improve layout
Parts:
- added C5: 100n, Capacitor_SMD:C_0805_2012Metric, B.Cu at (133.7, 116.0)
- moved R9 1.15 mm to (139.8, 116.0)
- moved R10 1.15 mm to (137.8, 116.0)
Routing:
- net Net-(J2-Pad2): track 5.31 -> 4.14 mm
- net Net-(J2-Pad3): track 5.69 -> 4.53 mm
- net /EXTINT: track 2.33 -> 3.19 mm
- net GND: vias 102 -> 103
- net +3V3: vias 2 -> 3
